Commit message: Método IK revisado
Se ha corregido la rotación de los vectores de referencia. Se estaba haciendo sobre los ejes de base_link. Esto es erróneo porque las rotaciones deben de aplicarse sobre los ejes locales. Se ha creado una nueva función encargada de rotar un vector según un eje local y un cierto ángulo.

File: urdf/human_right_arm_with_prismatic_joints.xacro (robot description, xacro)
@@ -1,25 +1,18 @@
 <?xml version="1.0"?>
-<!-- MODELO URDF DEL BRAZO HUMANO DERECHO -->
-<!-- Longitudes de los eslabones visuales parametrizadas con XACRO. Especificar en launch. -->
-<!-- Cuatro articulaciones de rotación [q1 q2 q3 q4] -->
-<!-- Articulaciones de la muñeca no se han considerado -->
-<!-- Contiene dos articulaciones prismáticas para adaptar las longitudes del brazo superior y del antebrazo. Esto afecta a TF -->
-<!-- ROS1 y RViz no permiten modificar el URDF de manera dinámica, luego, las longitudes de los eslabones visuales permanencen constante. Esto no afecta al calculo del Modelo Cinemático Directo -->
-<!-- Rodrigo Castro Ochoa, rcastro@uma.es, 2025-->
+<!-- Modelo del brazo derecho. Parametrizada con xacro-->
+<!-- Modelo con dos articulaciones prismaticas -->
+<!-- Opción 1. Diferencia visual acumulada en hombro y codo -->
 <robot xmlns:xacro="http://www.ros.org/wiki/xacro" name="human_right_arm">
-<!-- ############## Longitudes visuales parametrizadas ############## -->
+<!-- Longitudes parametrizadas -->
 <xacro:property name="visual_upperarm_length" value="$(arg visual_upperarm_length)"/>
 <xacro:property name="visual_forearm_length" value="$(arg visual_forearm_length)"/>
-<!-- ############## Color de los eslabones del URDF ############## -->
 <material name="color">
     <color rgba="0.1 0.1 0.1 1"/>
 </material>
-<!-- ############## ESLABONES ############## -->
-<!-- Los eslabones con f1 o f2 son eslabones ficticios. Unen articulaciones que se encuentran en un mismo punto -->
-<link name="base_shoulder"/> <!-- Base del URDF -->
+<link name="base_shoulder"/> <!-- Original del modelo URDF base. Sin embargo, no es util nuestro porque debería de estar alineado con el hombro. Alternativa: Considerar la siguiente TF como la inicial-->
 <link name="RightShoulder_f1" />
 <link name="RightShoulder_f2" />
 <link name="RightUpperArm_f1" />
-<link name="RightUpperArm"> <!-- Eslabón del upperarm -->
+<link name="RightUpperArm">
     <visual>
         <origin xyz="0 0 ${-visual_upperarm_length/2}" rpy="0 0 0"/>
@@ -32,5 +25,5 @@
 <link name="RightForeArm_f1" />
 <link name="RightForeArm_f2" />
-<link name="RightForeArm"> <!-- Eslabón del forearm -->
+<link name="RightForeArm">
     <visual>
         <origin xyz="0 0 ${-visual_forearm_length/2}" rpy="0 0 0"/>
@@ -41,5 +34,5 @@
     </visual>
 </link>
-<!-- Representación de la mano derecha -->
+<!-- Mano derecha -->
 <link name="RightFakeHand">
     <visual>
@@ -60,19 +53,19 @@
     </visual>
 </link>
-<!-- ############## ARTICULACIONES ############## -->
-<!-- Elevación frontal del hombro (q1) -->
+<!-- ARTICULACIONES -->
+<!-- Elevación del hombro (q1) -->
 <joint name="right_arm_q1" type="revolute">
     <origin xyz="0 0 0" rpy="1.5708 0 0"/>
     <parent link="base_shoulder"/>
     <child link="RightShoulder_f1"/>
-    <limit effort="30" velocity="1.0" lower="-0.5235987756" upper="2.61799387799"/> <!-- Límites articulares: -30º a 150º -->
+    <limit effort="30" velocity="1.0" lower="-0.5235987756" upper="2.61799387799"/> <!-- -30º a 150º -->
     <axis xyz="0 0 1"/> <!-- Rotación alrededor de Z -->
 </joint>
-<!-- Movimiento lateral del hombro (q2) -->
+<!-- Movimiento frontal del hombro (q2) -->
 <joint name="right_arm_q2" type="revolute">
     <origin xyz="0 0 0" rpy="0 -1.5708 0 "/> <!-- α = 90° -->
     <parent link="RightShoulder_f1"/>
     <child link="RightShoulder_f2"/>
-    <limit effort="30" velocity="1.0" lower="-0.5235987756" upper="2.26892802759"/> <!-- Límites articulares: -30º a 130º -->
+    <limit effort="30" velocity="1.0" lower="-0.5235987756" upper="2.26892802759"/> <!-- -30º a 130º -->
     <axis xyz="0 0 1"/> <!-- Rotación alrededor de Z -->
 </joint>
@@ -82,21 +75,21 @@
     <parent link="RightShoulder_f2"/>
     <child link="RightUpperArm_f1"/>
-    <limit effort="30" velocity="1.0" lower="0.1" upper="0.5"/> <!-- Límites articulares: 0.1m a 0.5m -->
-    <axis xyz="0 -1 0"/> <!-- Extensión en el eje Y (sentido negativo) -->
+    <limit effort="30" velocity="1.0" lower="0.1" upper="0.5"/> <!-- de 0.2m a 0.35m -->
+    <axis xyz="0 -1 0"/> <!-- Extensión en el eje Z -->
 </joint>
 <!-- Rotación interna/externa del hombro (q3) -->
 <joint name="right_arm_q3" type="revolute">
-    <origin xyz="0 0 0" rpy="1.5708 3.14159 0"/>
+    <origin xyz="0 0 0" rpy="1.5708 3.14159 0"/> <!-- d = 0.27m, α = 90° -->
     <parent link="RightUpperArm_f1"/>
     <child link="RightUpperArm"/>
-    <limit effort="30" velocity="1.0" lower="-1.57079632679" upper="1.57079632679"/> <!-- Límites articulares: -90° a 90°-->
+    <limit effort="30" velocity="1.0" lower="-1.57079632679" upper="1.57079632679"/> <!--  -90° a 90°-->
     <axis xyz="0 0 1"/> <!-- Rotación alrededor de Z -->
 </joint>
 <!-- Flexión del codo (q4) -->
 <joint name="right_arm_q4" type="revolute">
-    <origin xyz="0 0 0" rpy="1.5708 1.5708 0"/>
+    <origin xyz="0 0 0" rpy="1.5708 1.5708 0"/> <!-- d = -0.28m, α = -90°. Original: rpy="0 -1.5708 0" -->
     <parent link="RightUpperArm"/>
     <child link="RightForeArm_f1"/>
-    <limit effort="30" velocity="1.0" lower="0" upper="3.14159"/> <!-- Límites articulares: 0° a 180° -->
+    <limit effort="30" velocity="1.0" lower="0" upper="3.14159"/> <!-- 0° a 180° -->
     <axis xyz="0 0 1"/> <!-- Rotación alrededor de Z -->
 </joint>
@@ -106,16 +99,16 @@
     <parent link="RightForeArm_f1"/>
     <child link="RightForeArm_f2"/>
-    <limit effort="30" velocity="1.0" lower="0.1" upper="0.5"/> <!-- Límites articulares: de 0.1m a 0.5m -->
-    <axis xyz="1 0 0"/> <!-- Extensión en el eje X -->
+    <limit effort="30" velocity="1.0" lower="0.1" upper="0.5"/> <!-- de 0.2m a 0.35m -->
+    <axis xyz="1 0 0"/> <!-- Extensión en el eje Z -->
 </joint>
 <!-- Pronación/supinación del antebrazo (q5) -->
 <joint name="right_arm_q5" type="revolute">
-    <origin xyz="0 0 0" rpy="0 1.5708 0 "/>
+    <origin xyz="0 0 0" rpy="0 1.5708 0 "/> <!-- d = -0.25m, α = 90° -->
     <parent link="RightForeArm_f2"/>
     <child link="RightForeArm"/>
-    <limit effort="30" velocity="1.0" lower="0" upper="3.14159"/> <!-- Límites articulares: 0° a 180° -->
+    <limit effort="30" velocity="1.0" lower="0" upper="3.14159"/> <!-- 0° a 180° -->
     <axis xyz="0 0 1"/> <!-- Rotación alrededor de Z -->
 </joint>
-<!-- Articulaciones fijas de la mano. Entre los eslabones visuales de la mano. Se divide en dos partes -->
+<!-- Mano derecha. Se divide en dos partes -->
 <joint name="jRighthand_f1_fixed" type="fixed">
     <origin xyz="0 0 0.05" rpy="0 0 0 "/> <!-- l_box/ 2 -->
